Commit message: Feat: update TF node for moveit

File: isaac-ros/kistar_ws/src/franka_kistar_bringup/urdf/table.urdf.xacro (robot description, xacro)
@@ -35,5 +35,5 @@
   <link name="triangle_base">
     <visual>
-      <origin xyz="-0.185 -0.8 -0.75" rpy="0 0 0"/>
+      <origin xyz="-0.25 -0.8 -0.75" rpy="0 0 0"/>
       <geometry>
         <mesh filename="package://franka_kistar_bringup/meshes/table/triangle_1.STL" scale="0.001 0.001 0.001"/>
@@ -51,5 +51,5 @@
   <link name="triangle_base_2">
     <visual>
-      <origin xyz="-0.185 -0.8 -0.75" rpy="0 0 0"/>
+      <origin xyz="-0.25 -0.8 -0.75" rpy="0 0 0"/>
       <geometry>
         <mesh filename="package://franka_kistar_bringup/meshes/table/triangle_2.STL" scale="0.001 0.001 0.001"/>

File: isaac-ros/kistar_ws/src/franka_kistar_description/urdf/fr3_kistar.urdf.xacro (robot description, xacro)
@@ -39,5 +39,8 @@
     <parent link="fr3_link8"/>
     <child  link="kistar_hand"/>
-    <origin xyz="0 0 0" rpy="0 0 -0.785"/>
+    <!-- <origin xyz="0 0 0" rpy="0 0 -0.785"/> -->
+    <origin xyz="0 0 0" rpy="0 0 2.355"/>
   </joint>
+1
 </robot>
+    <!-- <origin xyz="0 0 0" rpy="0 0 -0.785"/> -->

File: isaac-ros/kistar_ws/src/franka_kistar_description/urdf/kistar_hand.xacro (robot description, xacro)
@@ -570,5 +570,6 @@
     </visual>
     <collision>
-      <origin xyz="0. 0. 0.02" rpy="0. 0. 0."/>
+      <!-- <origin xyz="0. 0. 0.02" rpy="0. 0. 0."/> -->
+      <origin xyz="0. 0. 0.05" rpy="0. 0. 0."/>
       <geometry>
         <box size="0.15 0.17 0.2"/>

Commit message: Fix: merge bug

File: isaac-ros/kistar_ws/src/franka_kistar_bringup/urdf/table.urdf.xacro (robot description, xacro)
@@ -35,9 +35,5 @@
   <link name="triangle_base">
     <visual>
-<<<<<<< HEAD
-      <origin xyz="-0.185 -0.8 -0.75" rpy="0 0 0"/>
-=======
       <origin xyz="-0.25 -0.8 -0.75" rpy="0 0 0"/>
->>>>>>> cy
       <geometry>
         <mesh filename="package://franka_kistar_bringup/meshes/table/triangle_1.STL" scale="0.001 0.001 0.001"/>
@@ -55,9 +51,5 @@
   <link name="triangle_base_2">
     <visual>
-<<<<<<< HEAD
       <origin xyz="-0.185 -0.8 -0.75" rpy="0 0 0"/>
-=======
-      <origin xyz="-0.25 -0.8 -0.75" rpy="0 0 0"/>
->>>>>>> cy
       <geometry>
         <mesh filename="package://franka_kistar_bringup/meshes/table/triangle_2.STL" scale="0.001 0.001 0.001"/>

File: isaac-ros/kistar_ws/src/franka_kistar_description/urdf/fr3_kistar.urdf.xacro (robot description, xacro)
@@ -39,12 +39,7 @@
     <parent link="fr3_link8"/>
     <child  link="kistar_hand"/>
-<<<<<<< HEAD
-    <origin xyz="0 0 0" rpy="0 0 -0.785"/>
-=======
     <!-- <origin xyz="0 0 0" rpy="0 0 -0.785"/> -->
     <origin xyz="0 0 0" rpy="0 0 2.355"/>
->>>>>>> cy
   </joint>
-1
 </robot>
     <!-- <origin xyz="0 0 0" rpy="0 0 -0.785"/> -->

File: isaac-ros/kistar_ws/src/franka_kistar_description/urdf/kistar_hand.xacro (robot description, xacro)
@@ -570,10 +570,6 @@
     </visual>
     <collision>
-<<<<<<< HEAD
-      <origin xyz="0. 0. 0.02" rpy="0. 0. 0."/>
-=======
       <!-- <origin xyz="0. 0. 0.02" rpy="0. 0. 0."/> -->
       <origin xyz="0. 0. 0.05" rpy="0. 0. 0."/>
->>>>>>> cy
       <geometry>
         <box size="0.15 0.17 0.2"/>
