Commit message: Feat: update hand collision mesh (fine)

File: isaac-ros/kistar_ws/src/franka_kistar_description/urdf/kistar_hand.xacro (robot description, xacro)
@@ -211,10 +211,10 @@
       </geometry>
     </visual>
-    <!-- <collision>
-      <origin xyz="0. -0. 0." rpy="0.0000013 0. 0. "/>
-      <geometry>
-        <mesh filename="package://franka_kistar_description/meshes/hand/index_basemotor_collisions.obj" scale="1. 1. 1."/>
-      </geometry> -->
-    <!-- </collision> -->
+    <collision>
+      <origin xyz="0.01407 0.0 0.0" rpy="0.0000013 0. 0."/>
+      <geometry>
+        <box size="0.02815 0.01920 0.02400"/>
+      </geometry>
+    </collision>
   </link>
   <link name="index_link_0">
@@ -230,10 +230,10 @@
       </geometry>
     </visual>
-    <!-- <collision>
-      <origin xyz="0. 0. 0." rpy="0. 0. 0."/>
-      <geometry>
-        <mesh filename="package://franka_kistar_description/meshes/hand/index_link_0_collisions.obj" scale="1. 1. 1."/>
-      </geometry>
-    </collision> -->
+    <collision>
+      <origin xyz="-0.00650 0.0 0.00977" rpy="0. 0. 0."/>
+      <geometry>
+        <box size="0.02600 0.02600 0.02845"/>
+      </geometry>
+    </collision>
   </link>
   <link name="index_link_1">
@@ -249,10 +249,10 @@
       </geometry>
     </visual>
-    <!-- <collision>
-      <origin xyz="0. 0. 0." rpy="0. 0. 0."/>
-      <geometry>
-        <mesh filename="package://franka_kistar_description/meshes/hand/index_link_1_collisions.obj" scale="1. 1. 1."/>
-      </geometry>
-    </collision> -->
+    <collision>
+      <origin xyz="-0.00162 0.0 0.01675" rpy="0. 0. 0."/>
+      <geometry>
+        <box size="0.01375 0.02610 0.04250"/>
+      </geometry>
+    </collision>
   </link>
   <link name="index_link_2">
@@ -268,10 +268,10 @@
       </geometry>
     </visual>
-    <!-- <collision>
-      <origin xyz="0. 0. 0." rpy="0. 0. 0."/>
-      <geometry>
-        <mesh filename="package://franka_kistar_description/meshes/hand/index_link_2_collisions.obj" scale="1. 1. 1."/>
-      </geometry>
-    </collision> -->
+    <collision>
+      <origin xyz="-0.00163 0.0 0.01335" rpy="0. 0. 0."/>
+      <geometry>
+        <box size="0.01375 0.02600 0.03570"/>
+      </geometry>
+    </collision>
   </link>
   <link name="index_tip">
@@ -287,10 +287,10 @@
       </geometry>
     </visual>
-    <!-- <collision>
-      <origin xyz="0. 0. -0." rpy="0. 0. 0."/>
-      <geometry>
-        <mesh filename="package://franka_kistar_description/meshes/hand/index_tip_collisions.obj" scale="1. 1. 1."/>
-      </geometry>
-    </collision> -->
+    <collision>
+      <origin xyz="-0.00200 0.0 0.01223" rpy="0. 0. 0."/>
+      <geometry>
+        <box size="0.01800 0.02600 0.03345"/>
+      </geometry>
+    </collision>
   </link>
   <link name="kistar_hand_index_sensor_0">
@@ -460,10 +460,10 @@
       </geometry>
     </visual>
-    <!-- <collision>
-      <origin xyz="0. 0. 0." rpy="0. 0. 0."/>
-      <geometry>
-        <mesh filename="package://franka_kistar_description/meshes/hand/middle_basemotor_collisions.obj" scale="1. 1. 1."/>
-      </geometry>
-    </collision> -->
+    <collision>
+      <origin xyz="0.01407 0.0 0.0" rpy="0. 0. 0."/>
+      <geometry>
+        <box size="0.02815 0.01920 0.02400"/>
+      </geometry>
+    </collision>
   </link>
   <link name="middle_link_0">
@@ -479,10 +479,10 @@
       </geometry>
     </visual>
-    <!-- <collision>
-      <origin xyz="0. 0. 0." rpy="0. 0. 0."/>
-      <geometry>
-        <mesh filename="package://franka_kistar_description/meshes/hand/middle_link_0_collisions.obj" scale="1. 1. 1."/>
-      </geometry>
-    </collision> -->
+    <collision>
+      <origin xyz="-0.00650 0.0 0.00977" rpy="0. 0. 0."/>
+      <geometry>
+        <box size="0.02600 0.02600 0.02845"/>
+      </geometry>
+    </collision>
   </link>
   <link name="middle_link_1">
@@ -498,10 +498,10 @@
       </geometry>
     </visual>
-    <!-- <collision>
-      <origin xyz="0. 0. 0." rpy="0. 0. 0."/>
-      <geometry>
-        <mesh filename="package://franka_kistar_description/meshes/hand/middle_link_1_collisions.obj" scale="1. 1. 1."/>
-      </geometry>
-    </collision> -->
+    <collision>
+      <origin xyz="-0.00162 0.0 0.01675" rpy="0. 0. 0."/>
+      <geometry>
+        <box size="0.01375 0.02610 0.04250"/>
+      </geometry>
+    </collision>
   </link>
   <link name="middle_link_2">
@@ -517,10 +517,10 @@
       </geometry>
     </visual>
-    <!-- <collision>
-      <origin xyz="0. 0. 0." rpy="0. 0. 0."/>
-      <geometry>
-        <mesh filename="package://franka_kistar_description/meshes/hand/middle_link_2_collisions.obj" scale="1. 1. 1."/>
-      </geometry>
-    </collision> -->
+    <collision>
+      <origin xyz="-0.00163 0.0 0.01335" rpy="0. 0. 0."/>
+      <geometry>
+        <box size="0.01375 0.02600 0.03570"/>
+      </geometry>
+    </collision>
   </link>
   <link name="middle_tip">
@@ -536,10 +536,10 @@
       </geometry>
     </visual>
-    <!-- <collision>
-      <origin xyz="0. 0. 0." rpy="0. 0. 0."/>
-      <geometry>
-        <mesh filename="package://franka_kistar_description/meshes/hand/middle_tip_collisions.obj" scale="1. 1. 1."/>
-      </geometry>
-    </collision> -->
+    <collision>
+      <origin xyz="-0.00200 0.0 0.01223" rpy="0. 0. 0."/>
+      <geometry>
+        <box size="0.01800 0.02600 0.03345"/>
+      </geometry>
+    </collision>
   </link>
   <link name="mount">
@@ -570,8 +570,7 @@
     </visual>
     <collision>
-      <!-- <origin xyz="0. 0. 0.02" rpy="0. 0. 0."/> -->
-      <origin xyz="0. 0. 0.05" rpy="0. 0. 0."/>
-      <geometry>
-        <box size="0.15 0.17 0.2"/>
+      <origin xyz="0.01070 0.0 -0.02702" rpy="0. 0. 0."/>
+      <geometry>
+        <box size="0.04700 0.08954 0.08512"/>
       </geometry>
     </collision>
@@ -589,10 +588,10 @@
       </geometry>
     </visual>
-    <!-- <collision>
-      <origin xyz="0. 0. 0." rpy="-0.0000013 0. 0. "/>
-      <geometry>
-        <mesh filename="package://franka_kistar_description/meshes/hand/ring_basemotor_collisions.obj" scale="1. 1. 1."/>
-      </geometry>
-    </collision> -->
+    <collision>
+      <origin xyz="0.01407 0.0 0.0" rpy="-0.0000013 0. 0."/>
+      <geometry>
+        <box size="0.02815 0.01920 0.02400"/>
+      </geometry>
+    </collision>
   </link>
   <link name="ring_link_0">
@@ -608,10 +607,10 @@
       </geometry>
     </visual>
-    <!-- <collision>
-      <origin xyz="0. 0. 0." rpy="0. 0. 0."/>
-      <geometry>
-        <mesh filename="package://franka_kistar_description/meshes/hand/ring_link_0_collisions.obj" scale="1. 1. 1."/>
-      </geometry>
-    </collision> -->
+    <collision>
+      <origin xyz="-0.00650 0.0 0.00977" rpy="0. 0. 0."/>
+      <geometry>
+        <box size="0.02600 0.02600 0.02845"/>
+      </geometry>
+    </collision>
   </link>
   <link name="ring_link_1">
@@ -627,10 +626,10 @@
       </geometry>
     </visual>
-    <!-- <collision>
-      <origin xyz="0. -0. 0." rpy="0. 0. 0."/>
-      <geometry>
-        <mesh filename="package://franka_kistar_description/meshes/hand/ring_link_1_collisions.obj" scale="1. 1. 1."/>
-      </geometry>
-    </collision> -->
+    <collision>
+      <origin xyz="-0.00162 0.0 0.01675" rpy="0. 0. 0."/>
+      <geometry>
+        <box size="0.01375 0.02610 0.04250"/>
+      </geometry>
+    </collision>
   </link>
   <link name="ring_link_2">
@@ -646,10 +645,10 @@
       </geometry>
     </visual>
-    <!-- <collision>
-      <origin xyz="0. -0. 0." rpy="0. 0. 0."/>
-      <geometry>
-        <mesh filename="package://franka_kistar_description/meshes/hand/ring_link_2_collisions.obj" scale="1. 1. 1."/>
-      </geometry>
-    </collision> -->
+    <collision>
+      <origin xyz="-0.00163 0.0 0.01335" rpy="0. 0. 0."/>
+      <geometry>
+        <box size="0.01375 0.02600 0.03570"/>
+      </geometry>
+    </collision>
   </link>
   <link name="ring_tip">
@@ -665,10 +664,10 @@
       </geometry>
     </visual>
-    <!-- <collision>
-      <origin xyz="0. -0. -0." rpy="0. 0. 0."/>
-      <geometry>
-        <mesh filename="package://franka_kistar_description/meshes/hand/ring_tip_collisions.obj" scale="1. 1. 1."/>
-      </geometry>
-    </collision> -->
+    <collision>
+      <origin xyz="-0.00200 0.0 0.01223" rpy="0. 0. 0."/>
+      <geometry>
+        <box size="0.01800 0.02600 0.03345"/>
+      </geometry>
+    </collision>
   </link>
   <link name="thumb_basemotor">
@@ -684,10 +683,10 @@
       </geometry>
     </visual>
-    <!-- <collision>
-      <origin xyz="0. 0. -0." rpy="0.0000013 0. 0. "/>
-      <geometry>
-        <mesh filename="package://franka_kistar_description/meshes/hand/thumb_basemotor_collisions.obj" scale="1. 1. 1."/>
-      </geometry>
-    </collision> -->
+    <collision>
+      <origin xyz="0.01200 0.0 0.0" rpy="0.0000013 0. 0."/>
+      <geometry>
+        <box size="0.02400 0.01920 0.02400"/>
+      </geometry>
+    </collision>
   </link>
   <link name="thumb_link_0">
@@ -703,10 +702,10 @@
       </geometry>
     </visual>
-    <!-- <collision>
-      <origin xyz="0. 0. 0." rpy="-0.0000013 0. 0. "/>
-      <geometry>
-        <mesh filename="package://franka_kistar_description/meshes/hand/thumb_link_0_collisions.obj" scale="1. 1. 1."/>
-      </geometry>
-    </collision> -->
+    <collision>
+      <origin xyz="-0.00716 0.0 0.01576" rpy="-0.0000013 0. 0."/>
+      <geometry>
+        <box size="0.02628 0.02600 0.04048"/>
+      </geometry>
+    </collision>
   </link>
   <link name="thumb_link_1">
@@ -722,10 +721,10 @@
       </geometry>
     </visual>
-    <!-- <collision>
-      <origin xyz="0. 0. 0." rpy="0. 0. 0."/>
-      <geometry>
-        <mesh filename="package://franka_kistar_description/meshes/hand/thumb_link_1_collisions.obj" scale="1. 1. 1."/>
-      </geometry>
-    </collision> -->
+    <collision>
+      <origin xyz="0.0 0.0 0.00724" rpy="0. 0. 0."/>
+      <geometry>
+        <box size="0.01300 0.02600 0.01448"/>
+      </geometry>
+    </collision>
   </link>
   <link name="thumb_link_2">
@@ -741,10 +740,10 @@
       </geometry>
     </visual>
-    <!-- <collision>
-      <origin xyz="0. 0. 0." rpy="0. 0. 0."/>
-      <geometry>
-        <mesh filename="package://franka_kistar_description/meshes/hand/thumb_link_2_collisions.obj" scale="1. 1. 1."/>
-      </geometry>
-    </collision> -->
+    <collision>
+      <origin xyz="-0.00162 0.0 0.01675" rpy="0. 0. 0."/>
+      <geometry>
+        <box size="0.01375 0.02610 0.04250"/>
+      </geometry>
+    </collision>
   </link>
   <link name="thumb_tip">
@@ -760,10 +759,10 @@
       </geometry>
     </visual>
-    <!-- <collision>
-      <origin xyz="0. 0. 0." rpy="0. 0. 0."/>
-      <geometry>
-        <mesh filename="package://franka_kistar_description/meshes/hand/thumb_tip_collisions.obj" scale="1. 1. 1."/>
-      </geometry>
-    </collision> -->
+    <collision>
+      <origin xyz="-0.00200 0.0 0.01223" rpy="0. 0. 0."/>
+      <geometry>
+        <box size="0.01800 0.02600 0.03345"/>
+      </geometry>
+    </collision>
   </link>
 </robot>
