Commit message: Feat: update moveit - isaac

File: isaac-ros/kistar_ws/src/franka_kistar_description/urdf/fr3_kistar.urdf.xacro (robot description, xacro)
@@ -1,7 +1,5 @@
 <?xml version="1.0"?>
 <robot name="fr3" xmlns:xacro="http://www.ros.org/wiki/xacro">
-  <!-- 1) 프랑카 공통 로봇 매크로 include -->
   <xacro:include filename="$(find franka_description)/robots/common/franka_robot.xacro"/>
-  <!-- 2) 우리가 expose 하고 싶은 arg만 다시 정의 (필요 최소한만) -->
   <xacro:arg name="arm_prefix"          default=""/>
   <xacro:arg name="ros2_control"        default="true"/>
@@ -10,18 +8,5 @@
   <xacro:arg name="fake_sensor_commands" default="false"/>
   <xacro:property name="arm_id" value="fr3"/>
-  <xacro:arg name="safety_distance" default="0.03" />
-  <xacro:arg name="with_sc" default="false" />
-  <xacro:arg name="arm_id" default="fr3" />
-  <xacro:arg name="no_prefix" default="false"/>
-  <!-- <xacro:arg name="hand" default="true" /> -->
-  <!-- <xacro:arg name="ee_id" default="franka_hand" /> -->
-  <xacro:arg name="special_connection" default="" />
-  <xacro:arg name="xyz_ee" default="0 0 0" />
-  <xacro:arg name="rpy_ee" default= "0 0 ${-pi/4}" />
-  <xacro:arg name="tcp_xyz" default="0 0 0.1034" />
-  <xacro:arg name="tcp_rpy" default="0 0 0" />
-  <xacro:property name="arm_prefix_val" value="$(arg arm_prefix)"/>
   <xacro:property name="flange_link" value="${arm_prefix_val + arm_id + '_link8'}"/>
-  <!-- 3) 프랑카 팔만 생성: hand= false, ee_id= none 으로 기본 그리퍼 끄기 -->
   <xacro:franka_robot
       arm_id="fr3"
@@ -38,6 +23,6 @@
       rpy_ee="0 0 0"
       tcp_xyz="0 0 0.1034"
-      tcp_rpy="0 0 0"
-      safety_distance="0.0"
+      tcp_rpy="0.0 0 0"
+      safety_distance="0.03"
       with_sc="false"
       ros2_control="$(arg ros2_control)"
@@ -52,5 +37,4 @@
   <xacro:include filename="$(find franka_kistar_description)/urdf/kistar_hand.xacro"/>
   <joint name="kistar_hand_mount" type="fixed">
-    <!-- <parent link="${flange_link}"/> -->
     <parent link="fr3_link8"/>
     <child  link="kistar_hand"/>

File: isaac-ros/kistar_ws/src/franka_kistar_description/urdf/kistar_hand.xacro (robot description, xacro)
@@ -769,19 +769,19 @@
   <link name="lab_table">
     <visual>
-      <origin xyz="0.5 0.0 -0.36" rpy="0 0 0"/>
-      <geometry>
-        <!-- size: x(길이) y(폭) z(높이) -->
-        <box size="1.0 0.6 0.72"/>
-      </geometry>
-      <material name="lab_table_color">
-        <color rgba="0.6 0.4 0.3 1.0"/>
-      </material>
+      <origin xyz="-0.25 -1.1 -0.15" rpy="-0.785 0 0"/>
+      <geometry>
+        <mesh filename="package://franka_kistar_description/meshes/table/soldering_table.obj" scale="1. 1. 1."/>
+      </geometry>
     </visual>
     <collision>
       <!-- 충돌 모델도 동일 박스 -->
-      <origin xyz="0.5 0.0 -0.36" rpy="0 0 0"/>
+      <!-- <origin xyz="0.5 0.0 -0.36" rpy="-0.785 0 0"/>
       <geometry>
         <box size="1.0 0.6 0.72"/>
-      </geometry>
+      </geometry> -->
+        <origin xyz="-0.25 -1.1 -0.15" rpy="-0.785 0 0"/>
+        <geometry>
+          <mesh filename="package://franka_kistar_description/meshes/table/soldering_table.obj" scale="1. 1. 1."/>
+        </geometry>
     </collision>
   </link>

Commit message: Feat: just backup

File: isaac-ros/kistar_ws/src/franka_kistar_description/urdf/fr3_kistar.urdf.xacro (robot description, xacro)
@@ -16,5 +16,5 @@
       accelerometer_config="${xacro.load_yaml('$(find franka_kistar_description)/robots/fr3/accelerometers.yaml')}"
       dynamics="${xacro.load_yaml('$(find franka_kistar_description)/robots/fr3/dynamics.yaml')}"
-      gazebo="true"
+      gazebo="false"
       hand="false"
       ee_id="none"

File: isaac-ros/kistar_ws/src/franka_kistar_description/urdf/kistar_hand_bck.xacro (robot description, xacro)
@@ -767,3 +767,26 @@
     </collision> -->
   </link>
+  <link name="lab_table">
+    <visual>
+      <origin xyz="-0.25 -1.1 -0.15" rpy="-0.785 0 0"/>
+      <geometry>
+        <mesh filename="package://franka_kistar_description/meshes/table/soldering_table.obj" scale="1. 1. 1."/>
+      </geometry>
+    </visual>
+    <collision>
+      <!-- 충돌 모델도 동일 박스 -->
+      <!-- <origin xyz="0.5 0.0 -0.36" rpy="-0.785 0 0"/>
+      <geometry>
+        <box size="1.0 0.6 0.72"/>
+      </geometry> -->
+        <origin xyz="-0.25 -1.1 -0.15" rpy="-0.785 0 0"/>
+        <geometry>
+          <mesh filename="package://franka_kistar_description/meshes/table/soldering_table.obj" scale="1. 1. 1."/>
+        </geometry>
+    </collision>
+  </link>
+  <joint name="lab_table_fixed" type="fixed">
+    <parent link="fr3_link0"/>
+    <child  link="lab_table"/>
+  </joint>
 </robot>

Commit message: Feat: update TF Setting and Docs

File: isaac-ros/kistar_ws/src/franka_kistar_description/urdf/fr3_kistar.urdf.xacro (robot description, xacro)
@@ -39,4 +39,5 @@
     <parent link="fr3_link8"/>
     <child  link="kistar_hand"/>
+    <origin xyz="0 0 0" rpy="0 0 -0.785"/>
   </joint>
 </robot>

File: isaac-ros/kistar_ws/src/franka_kistar_description/urdf/kistar_hand.xacro (robot description, xacro)
@@ -51,5 +51,4 @@
   </joint>
   <joint name="kistar_mount_joint" type="fixed">
-    <!-- <origin xyz="-0.02325 0. 0.071 " rpy="0. 0. 0."/> -->
     <origin xyz="-0.01 0. 0.071 " rpy="0. 0. 0."/>
     <parent link="mount"/>
@@ -571,7 +570,7 @@
     </visual>
     <collision>
-      <origin xyz="0. 0. 0." rpy="0. 0. 45."/>
-      <geometry>
-        <mesh filename="package://franka_kistar_description/meshes/hand/fr3_hand_collisions.obj" scale="5 1.5 3"/>
+      <origin xyz="0. 0. 0.02" rpy="0. 0. 0."/>
+      <geometry>
+        <box size="0.15 0.17 0.2"/>
       </geometry>
     </collision>

Commit message: Cy (#3)
* Feat: update - humble python11 ros2 version

* backup

* Feat: Just add skeleton for kistar launch

* Feat: add franka-kistar ros2 package for moveit

* Feat: update ros2-isaac and ros2-moveit

* Feat: update moveit - isaac

* Feat: update docs..

* Docs: update moveit example!

* Add: gitignore

* Feat: remove test file

* Docs: update quick start

* Feat: update

* Docs: update sim-moveit commands.

* Feat: Add real-moveit launch + bridge

* Feat: update district movement

* Feat update

* Feat update

* Feat update

* Feat: generate smooth movement with moveit

* Docs: update develop status

* Docs: update additional explanation

* Feat: just backup

* Feat: update TF Setting and Docs

* Docs: update docs

File: isaac-ros/kistar_ws/src/franka_kistar_description/urdf/fr3_kistar.urdf.xacro (robot description, xacro)
@@ -16,5 +16,5 @@
       accelerometer_config="${xacro.load_yaml('$(find franka_kistar_description)/robots/fr3/accelerometers.yaml')}"
       dynamics="${xacro.load_yaml('$(find franka_kistar_description)/robots/fr3/dynamics.yaml')}"
-      gazebo="true"
+      gazebo="false"
       hand="false"
       ee_id="none"
@@ -39,4 +39,5 @@
     <parent link="fr3_link8"/>
     <child  link="kistar_hand"/>
+    <origin xyz="0 0 0" rpy="0 0 -0.785"/>
   </joint>
 </robot>

File: isaac-ros/kistar_ws/src/franka_kistar_description/urdf/kistar_hand.xacro (robot description, xacro)
@@ -51,5 +51,4 @@
   </joint>
   <joint name="kistar_mount_joint" type="fixed">
-    <!-- <origin xyz="-0.02325 0. 0.071 " rpy="0. 0. 0."/> -->
     <origin xyz="-0.01 0. 0.071 " rpy="0. 0. 0."/>
     <parent link="mount"/>
@@ -571,7 +570,7 @@
     </visual>
     <collision>
-      <origin xyz="0. 0. 0." rpy="0. 0. 45."/>
-      <geometry>
-        <mesh filename="package://franka_kistar_description/meshes/hand/fr3_hand_collisions.obj" scale="5 1.5 3"/>
+      <origin xyz="0. 0. 0.02" rpy="0. 0. 0."/>
+      <geometry>
+        <box size="0.15 0.17 0.2"/>
       </geometry>
     </collision>
@@ -767,26 +766,3 @@
     </collision> -->
   </link>
-  <link name="lab_table">
-    <visual>
-      <origin xyz="-0.25 -1.1 -0.15" rpy="-0.785 0 0"/>
-      <geometry>
-        <mesh filename="package://franka_kistar_description/meshes/table/soldering_table.obj" scale="1. 1. 1."/>
-      </geometry>
-    </visual>
-    <collision>
-      <!-- 충돌 모델도 동일 박스 -->
-      <!-- <origin xyz="0.5 0.0 -0.36" rpy="-0.785 0 0"/>
-      <geometry>
-        <box size="1.0 0.6 0.72"/>
-      </geometry> -->
-        <origin xyz="-0.25 -1.1 -0.15" rpy="-0.785 0 0"/>
-        <geometry>
-          <mesh filename="package://franka_kistar_description/meshes/table/soldering_table.obj" scale="1. 1. 1."/>
-        </geometry>
-    </collision>
-  </link>
-  <joint name="lab_table_fixed" type="fixed">
-    <parent link="fr3_link0"/>
-    <child  link="lab_table"/>
-  </joint>
 </robot>

Commit message: GWB ver update

File: isaac-ros/kistar_ws/src/franka_kistar_description/urdf/fr3_kistar.urdf.xacro (robot description, xacro)
@@ -8,5 +8,4 @@
   <xacro:arg name="fake_sensor_commands" default="false"/>
   <xacro:property name="arm_id" value="fr3"/>
-  <xacro:property name="flange_link" value="${arm_prefix_val + arm_id + '_link8'}"/>
   <xacro:franka_robot
       arm_id="fr3"
@@ -14,5 +13,4 @@
       inertials="${xacro.load_yaml('$(find franka_kistar_description)/robots/fr3/inertials.yaml')}"
       kinematics="${xacro.load_yaml('$(find franka_kistar_description)/robots/fr3/kinematics.yaml')}"
-      accelerometer_config="${xacro.load_yaml('$(find franka_kistar_description)/robots/fr3/accelerometers.yaml')}"
       dynamics="${xacro.load_yaml('$(find franka_kistar_description)/robots/fr3/dynamics.yaml')}"
       gazebo="false"
